File: PSFB_Supply/PSFB_Supply.kicad_pcb (KiCad board)
At the start: 2 copper layers, 43 x 74 mm, 36 parts, among them J1 PWR_IN, J2 PWR_IN, J3 PWR_IN, J4 PWR_IN, J5 PWR_IN, J6 PWR_IN

Commit message: VER1.0: добавил интерактивный BOM
Parts:
- D1, D2, D3, D4: value QA151C3 -> ~
- J1, J2, J3, J4, J5, J6: value PWR_IN -> ~
