File: PSFB_Supply/QA01.kicad_sch (KiCad schematic)
At the start: 8 parts, among them J1 PWR_IN

Commit message: VER1.0: добавил интерактивный BOM
Parts:
- C1, C2, C3, C4, C5: Description P/N (none) -> Capacitor SMD 50V
- D1: value QA151C3 -> (none); Description P/N (none) -> DC/DC; Product Name (none) -> QA151C3
- J1: value PWR_IN -> (none); Description P/N (none) -> Connector; Product Name (none) -> KLS1-207-2-04-S
- L1: Description P/N (none) -> Inductor SMD; Product Name (none) -> CDRH5D28NP-220NC
Changed lines of the file:
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@@
+			)
+		)
+		(property "Description P/N" "Capacitor SMD 50V"
+			(at 168.91 86.36 0)
+			(hide yes)
+			(show_name no)
+			(do_not_autoplace no)
+			(effects
+				(font
+					(size 1.27 1.27)
+				)
 			)
 		)
@@
 			)
 		)
+		(property "Description P/N" "Capacitor SMD 50V"
+			(at 119.38 90.17 0)
+			(hide yes)
+			(show_name no)
+			(do_not_autoplace no)
+			(effects
+				(font
+					(size 1.27 1.27)
+				)
+			)
+		)
 		(pin "1"
 		)
@@
 		)
 		(property "Description" "Unpolarized capacitor, small symbol"
+			(at 168.91 93.98 0)
+			(hide yes)
+			(show_name no)
+			(do_not_autoplace no)
+			(effects
+				(font
+					(size 1.27 1.27)
+				)
+			)
+		)
+		(property "Description P/N" "Capacitor SMD 50V"
 			(at 168.91 93.98 0)
 			(hide yes)
@@
 			)
 		)
-		(property "Value" "QA151C3"
+		(property "Value" ""
 			(at 143.51 82.55 0)
 			(show_name no)
@@
 		)
 		(property "Description" ""
+			(at 143.51 90.17 0)
+			(hide yes)
+			(show_name no)
+			(do_not_autoplace no)
+			(effects
+				(font
+					(size 1.27 1.27)
+				)
+			)
+		)
+		(property "Product Name" "QA151C3"
+			(at 143.51 90.17 0)
+			(hide yes)
+			(show_name no)
+			(do_not_autoplace no)
+			(effects
+				(font
+					(size 1.27 1.27)
+				)
+			)
+		)
+		(property "Description P/N" "DC/DC"
 			(at 143.51 90.17 0)
 			(hide yes)
@@
 			)
 		)
+		(property "Description P/N" "Capacitor SMD 50V"
+			(at 107.95 90.17 0)
+			(hide yes)
+			(show_name no)
+			(do_not_autoplace no)
+			(effects
+				(font
+					(size 1.27 1.27)
+				)
+			)
+		)
 		(pin "1"
 		)
@@
 			)
 		)
-		(property "Datasheet" "CDRH5D28NP-220NC"
+		(property "Datasheet" ""
 			(at 114.3 87.63 0)
 			(hide yes)
@@
 		)
 		(property "Description" "Inductor, small symbol"
+			(at 114.3 87.63 0)
+			(hide yes)
+			(show_name no)
+			(do_not_autoplace no)
+			(effects
+				(font
+					(size 1.27 1.27)
+				)
+			)
+		)
+		(property "Product Name" "CDRH5D28NP-220NC"
+			(at 114.3 87.63 0)
+			(hide yes)
+			(show_name no)
+			(do_not_autoplace no)
+			(effects
+				(font
+					(size 1.27 1.27)
+				)
+			)
+		)
+		(property "Description P/N" "Inductor SMD"
+			(at 114.3 87.63 0)
+			(hide yes)
+			(show_name no)
+			(do_not_autoplace no)
+			(effects
+				(font
+					(size 1.27 1.27)
+				)
+			)
+		)
+		(property "Replacement" ""
+			(at 114.3 87.63 0)
+			(hide yes)
+			(show_name no)
+			(do_not_autoplace no)
+			(effects
+				(font
+					(size 1.27 1.27)
+				)
+			)
+		)
+		(property "Function" ""
 			(at 114.3 87.63 0)
 			(hide yes)
@@
 		)
 		(property "Description" "Unpolarized capacitor, small symbol"
+			(at 125.73 90.17 0)
+			(hide yes)
+			(show_name no)
+			(do_not_autoplace no)
+			(effects
+				(font
+					(size 1.27 1.27)
+				)
+			)
+		)
+		(property "Description P/N" "Capacitor SMD 50V"
 			(at 125.73 90.17 0)
 			(hide yes)
@@
 			)
 		)
-		(property "Value" "PWR_IN"
+		(property "Value" ""
 			(at 176.53 88.9 0)
 			(hide yes)
@@
 			(at 180.34 90.17 0)
 			(hide yes)
+			(show_name no)
+			(do_not_autoplace no)
+			(effects
+				(font
+					(size 1.27 1.27)
+				)
+			)
+		)
+		(property "Product Name" "KLS1-207-2-04-S"
+			(at 180.34 90.17 0)
+			(hide yes)
+			(show_name no)
+			(do_not_autoplace no)
+			(effects
+				(font
+					(size 1.27 1.27)
+				)
+			)
+		)
+		(property "Description P/N" "Connector"
+			(at 180.34 90.17 0)
+			(hide yes)
+			(show_name no)
+			(do_not_autoplace no)
+			(effects
+				(font
+					(size 1.27 1.27)
+				)
+			)
+		)
+		(property "Replacement" ""
+			(at 180.34 90.17 0)
+			(hide yes)
+			(show_name no)
+			(do_not_autoplace no)
+			(effects
+				(font
+					(size 1.27 1.27)
+				)
+			)
+		)
+		(property "Function" ""
+			(at 180.34 90.17 0)
+			(hide yes)
